File: V3/Full.brd (EAGLE design)
At the start: 246.4 x 317.5 mm, 236 parts, among them X1 SSW-103-02-G-S

Commit message: Commit xD
Parts:
- CLOCK: value (none) -> Yellow
- RESET_PC, RESET_REGS: value (none) -> NORM-OFF
Routing:
- net GND: track 426.4 -> 440.1 mm
Changed lines of the file:
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@@
 <attribute name="VALUE" x="42.672" y="284.48" size="1.27" layer="27" ratio="10"/>
 </element>
-<element name="CLOCK" library="led" library_urn="urn:adsk.eagle:library:259" package="LED5MM" package3d_urn="urn:adsk.eagle:package:15799/2" value="" x="60.96" y="289.56" smashed="yes">
+<element name="CLOCK" library="led" library_urn="urn:adsk.eagle:library:259" package="LED5MM" package3d_urn="urn:adsk.eagle:package:15799/2" value="Yellow" x="60.96" y="289.56" smashed="yes">
 <attribute name="NAME" x="57.785" y="283.7434" size="1.27" layer="25" ratio="10"/>
 <attribute name="POPULARITY" value="93" x="99.06" y="53.34" size="1.778" layer="27" display="off"/>
@@
 <attribute name="VALUE" x="13.335" y="52.959" size="1.27" layer="27" ratio="10"/>
 </element>
-<element name="RESET_PC" library="switch-omron" library_urn="urn:adsk.eagle:library:377" package="B3F-10XX" package3d_urn="urn:adsk.eagle:package:27496/1" value="" x="170.18" y="300.99" smashed="yes">
+<element name="RESET_PC" library="switch-omron" library_urn="urn:adsk.eagle:library:377" package="B3F-10XX" package3d_urn="urn:adsk.eagle:package:27496/1" value="NORM-OFF" x="170.18" y="300.99" smashed="yes">
 <attribute name="MF" value="" x="347.98" y="100.33" size="1.778" layer="27" display="off"/>
 <attribute name="MPN" value="B3F-1000" x="347.98" y="100.33" size="1.778" layer="27" display="off"/>
@@
 <attribute name="VALUE" x="167.132" y="295.91" size="1.27" layer="27" ratio="10"/>
 </element>
-<element name="RESET_REGS" library="switch-omron" library_urn="urn:adsk.eagle:library:377" package="B3F-10XX" package3d_urn="urn:adsk.eagle:package:27496/1" value="" x="105.41" y="190.5" smashed="yes">
+<element name="RESET_REGS" library="switch-omron" library_urn="urn:adsk.eagle:library:377" package="B3F-10XX" package3d_urn="urn:adsk.eagle:package:27496/1" value="NORM-OFF" x="105.41" y="190.5" smashed="yes">
 <attribute name="MF" value="" x="270.51" y="-10.16" size="1.778" layer="27" display="off"/>
 <attribute name="MPN" value="B3F-1000" x="270.51" y="-10.16" size="1.778" layer="27" display="off"/>
@@
 <wire x1="15.24" y1="167.64" x2="21.3106" y2="161.5694" width="0.1524" layer="1"/>
 <wire x1="21.3106" y1="161.5694" x2="21.3106" y2="160.9217625" width="0.1524" layer="1"/>
-<wire x1="22.86" y1="159.3723625" x2="22.86" y2="158.75" width="0.1524" layer="1"/>
-<wire x1="21.3106" y1="160.9217625" x2="22.86" y2="159.3723625" width="0.1524" layer="1"/>
 <via x="31.75" y="152.4" extent="1-16" drill="0.35"/>
 <wire x1="26.9113625" y1="151.511" x2="28.9686375" y2="151.511" width="0.1524" layer="1"/>
@@
 <wire x1="31.75" y1="152.4" x2="31.75" y2="154.94" width="0.1524" layer="16"/>
 <via x="31.75" y="154.94" extent="1-16" drill="0.35"/>
-<wire x1="22.86" y1="158.1276375" x2="22.86" y2="158.75" width="0.1524" layer="1"/>
 <wire x1="35.56" y1="21.59" x2="38.1" y2="21.59" width="0.1524" layer="1"/>
 <via x="38.1" y="21.59" extent="1-16" drill="0.35"/>
@@
 <wire x1="165.1" y1="232.41" x2="166.37" y2="233.68" width="0.1524" layer="16"/>
 <via x="166.37" y="233.68" extent="1-16" drill="0.35"/>
+<wire x1="21.3106" y1="166.7382375" x2="21.8313625" y2="167.259" width="0.1524" layer="1"/>
+<wire x1="21.8313625" y1="167.259" x2="23.8886375" y2="167.259" width="0.1524" layer="1"/>
+<wire x1="23.8886375" y1="167.259" x2="24.4094" y2="166.7382375" width="0.1524" layer="1"/>
+<wire x1="22.86" y1="158.75" x2="22.86" y2="159.3723625" width="0.1524" layer="1"/>
+<wire x1="22.86" y1="159.3723625" x2="21.3106" y2="160.9217625" width="0.1524" layer="1"/>
+<wire x1="24.4094" y1="166.7382375" x2="24.4094" y2="166.0906" width="0.1524" layer="1"/>
+<wire x1="24.4094" y1="166.0906" x2="27.94" y2="162.56" width="0.1524" layer="1"/>
+<wire x1="21.3106" y1="161.5694" x2="21.3106" y2="166.7382375" width="0.1524" layer="1"/>
 </signal>
 <signal name="VCC">

Commit message: Tidy and added Instructions
Connections:
- new net N$232: ADDER_UPPER.9, XOR_GATE_2.12
- net CTRL_SIG_12: now also XOR_GATE_2.13
- net OVERFLOW_FLAG: now also XOR_GATE_2.11; no longer ADDER_UPPER.9
Routing:
- net OVERFLOW_FLAG: track 315.0 -> 302.4 mm
Changed lines of the file:
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@@
 </signal>
 <signal name="OVERFLOW_FLAG">
-<contactref element="ADDER_UPPER" pad="9"/>
 <contactref element="FLAG_REG_LOWER" pad="14"/>
 <contactref element="OVERFLOW_FLAG" pad="A"/>
@@
 <wire x1="135.255" y1="236.855" x2="135.255" y2="203.835" width="0.1524" layer="16"/>
 <wire x1="135.255" y1="237.49" x2="135.255" y2="236.855" width="0.1524" layer="1"/>
-<wire x1="199.39" y1="240.03" x2="208.28" y2="231.14" width="0.1524" layer="1"/>
 <wire x1="169.545" y1="240.03" x2="199.39" y2="240.03" width="0.1524" layer="1"/>
 <wire x1="166.37" y1="236.855" x2="169.545" y2="240.03" width="0.1524" layer="16"/>
@@
 <via x="135.255" y="236.855" extent="1-16" drill="0.35"/>
 <via x="169.545" y="240.03" extent="1-16" drill="0.35"/>
+<contactref element="XOR_GATE_2" pad="11"/>
+<wire x1="121.92" y1="26.67" x2="119.38" y2="19.05" width="0" layer="19" extent="1-1"/>
 </signal>
 <signal name="N$58">
@@
 <wire x1="200.66" y1="204.47" x2="202.565" y2="206.375" width="0.1524" layer="1"/>
 <via x="52.705" y="200.025" extent="1-16" drill="0.35"/>
+<contactref element="XOR_GATE_2" pad="13"/>
+<wire x1="114.3" y1="19.05" x2="43.18" y2="124.46" width="0" layer="19" extent="1-1"/>
 </signal>
 <signal name="MICRO_A8">
@@
 <via x="119.38" y="238.76" extent="1-16" drill="0.35"/>
 </signal>
+<signal name="N$232">
+<contactref element="ADDER_UPPER" pad="9"/>
+<contactref element="XOR_GATE_2" pad="12"/>
+<wire x1="116.84" y1="19.05" x2="208.28" y2="231.14" width="0" layer="19" extent="1-1"/>
+</signal>
 </signals>

Commit message: Updated spreadsheet and overwritten XOR gate for overflow on subtract
Connections:
- removed net N$232: ADDER_UPPER.9, XOR_GATE_2.12
- net CTRL_SIG_12: no longer XOR_GATE_2.13
- net OVERFLOW_FLAG: now also ADDER_UPPER.9; no longer XOR_GATE_2.11
Changed lines of the file:
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@@
 <via x="135.255" y="236.855" extent="1-16" drill="0.35"/>
 <via x="169.545" y="240.03" extent="1-16" drill="0.35"/>
-<contactref element="XOR_GATE_2" pad="11"/>
-<wire x1="121.92" y1="26.67" x2="119.38" y2="19.05" width="0" layer="19" extent="1-1"/>
+<contactref element="ADDER_UPPER" pad="9"/>
+<wire x1="199.39" y1="240.03" x2="208.28" y2="231.14" width="0" layer="19" extent="1-1"/>
 </signal>
 <signal name="N$58">
@@
 <wire x1="200.66" y1="204.47" x2="202.565" y2="206.375" width="0.1524" layer="1"/>
 <via x="52.705" y="200.025" extent="1-16" drill="0.35"/>
-<contactref element="XOR_GATE_2" pad="13"/>
-<wire x1="114.3" y1="19.05" x2="43.18" y2="124.46" width="0" layer="19" extent="1-1"/>
 </signal>
 <signal name="MICRO_A8">
@@
 <via x="119.38" y="238.76" extent="1-16" drill="0.35"/>
 </signal>
-<signal name="N$232">
-<contactref element="ADDER_UPPER" pad="9"/>
-<contactref element="XOR_GATE_2" pad="12"/>
-<wire x1="116.84" y1="19.05" x2="208.28" y2="231.14" width="0" layer="19" extent="1-1"/>
-</signal>
 </signals>
