File: V4/Full.brd (EAGLE design)
At the start: 246.4 x 317.5 mm, 206 parts, among them X1 SSW-103-02-G-S

Commit message: update
Parts:
- added INP_SELECTOR: 74AC139N, 74xx-eu:DIL16
- moved SELECTOR_RAM_ 85.3 mm to (73.7, 53.3), turned to 270 degrees
Connections:
- new net N$40: INP_SELECTOR.3, INSTRUCTION_MEMORY_2.16
- new net N$56: INP_SELECTOR.2, INSTRUCTION_MEMORY_2.17
- net CTRL_SIG_21_(P_REG_IN): now also INP_SELECTOR.6; no longer INSTRUCTION_MEMORY_2.16
- net CTRL_SIG_22_(P_REG_OUT): now also INP_SELECTOR.5; no longer INSTRUCTION_MEMORY_2.17
- net GND: now also INP_SELECTOR.1, INP_SELECTOR.8
- net VCC: now also INP_SELECTOR.16
Routing:
- net GND: track 431.5 -> 0.00 mm, vias 41 -> 0
- net VCC: track 252.6 -> 0.00 mm, vias 22 -> 0
- net PC_OUT: track 70.2 -> 306.6 mm
- net N$212: track 314.6 -> 95.4 mm, vias 3 -> 0
- net N$55: track 278.1 -> 72.1 mm, vias 4 -> 1
- net REG_B_8PLACE: track 371.7 -> 205.1 mm, vias 5 -> 2
- net N$26: track 0.00 -> 160.1 mm, vias 0 -> 1
- net PC_LOAD_SIGNAL: track 91.9 -> 242.9 mm, vias 0 -> 3
- net N$10: track 0.00 -> 133.7 mm, vias 0 -> 2
- net N$56: track 0.00 -> 113.7 mm, vias 0 -> 1
- net N$40: track 0.00 -> 106.4 mm, vias 0 -> 1
- net 1_PLACE: track 995.7 -> 891.4 mm, vias 9 -> 15
- net REG_A_1PLACE: track 252.6 -> 149.6 mm, vias 5 -> 2
- net REG_A_128PLACE: track 264.2 -> 171.6 mm, vias 3 -> 4
- net REG_A_32PLACE: track 264.7 -> 172.2 mm, vias 5 -> 2
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Other:
- board text removed: "AND"
- board text removed: "NOT"
- board text removed: "OR"
- board text removed: "Selector Combines"
- board text removed: "XOR"
