File: V4/Full.brd (EAGLE design)
At the start: 246.4 x 317.5 mm, 216 parts, among them IC1 74LS595N, IC2 74LS595N, IC4 74LS02N, IC5 74S86N, X1 SSW-103-02-G-S

Commit message: update
Parts:
- added D1: 1N4728, diode:DO41Z10
Connections:
- net N$106: now also D1.C
- net N$63: now also D1.A
Changed lines of the file:
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@@
 <layer number="97" name="Info" color="7" fill="1" visible="no" active="no"/>
 <layer number="98" name="Guide" color="6" fill="1" visible="no" active="no"/>
+<layer number="99" name="SpiceOrder" color="5" fill="1" visible="no" active="no"/>
 </layers>
 <board>
@@
 <attribute name="VALUE" x="3.429" y="-114.935" size="1.27" layer="27" ratio="10"/>
 </element>
+<element name="D1" library="diode" library_urn="urn:adsk.eagle:library:210" package="DO41Z10" package3d_urn="urn:adsk.eagle:package:43341/1" value="1N4728" x="5.08" y="-123.19" smashed="yes">
+<attribute name="NAME" x="3.175" y="-121.539" size="1.27" layer="25" ratio="10"/>
+<attribute name="POPULARITY" value="6" x="5.08" y="-123.19" size="1.778" layer="27" display="off"/>
+<attribute name="VALUE" x="3.175" y="-125.984" size="1.27" layer="27" ratio="10"/>
+</element>
 </elements>
 <signals>
@@
 <contactref element="NOT_GATE3_" pad="5"/>
 <contactref element="R6" pad="1"/>
+<contactref element="D1" pad="A"/>
 <wire x1="140.97" y1="242.57" x2="140.97" y2="250.19" width="0" layer="19" extent="1-1"/>
 <wire x1="15.24" y1="-24.13" x2="140.97" y2="242.57" width="0" layer="19" extent="1-1"/>
 <wire x1="15.24" y1="-35.56" x2="15.24" y2="-24.13" width="0" layer="19" extent="1-1"/>
 <wire x1="0" y1="-88.9" x2="15.24" y2="-35.56" width="0" layer="19" extent="1-1"/>
+<wire x1="10.16" y1="-123.19" x2="0" y2="-88.9" width="0" layer="19" extent="1-1"/>
 </signal>
 <signal name="N$81">
@@
 <contactref element="NOT_GATE_" pad="3"/>
 <contactref element="IC4" pad="3"/>
+<contactref element="D1" pad="C"/>
 <wire x1="7.62" y1="-88.9" x2="125.73" y2="257.81" width="0" layer="19" extent="1-1"/>
 <wire x1="1.524" y1="-93.98" x2="7.62" y2="-88.9" width="0" layer="19" extent="1-1"/>
 <wire x1="7.62" y1="-106.68" x2="1.524" y2="-93.98" width="0" layer="19" extent="1-1"/>
+<wire x1="0" y1="-123.19" x2="7.62" y2="-106.68" width="0" layer="19" extent="1-1"/>
 </signal>
 <signal name="N$108">

Commit message: update
Parts:
- removed IC3: (no value), ic-package:DIL28-6
- removed IC5: 74S86N, 74xx-eu:DIL14
- removed INP_SELECTOR: 74AC139N, 74xx-eu:DIL16
- added FIFO_STACK: 71256SA15TPG, ic-package:DIL28-3
- added OUTPUT_BUFFER_KEYBOARD: 74LS245N, 74xx-eu:DIL20
- added OUT_REG_LOWER, OUT_REG_UPPER: 74LS173N, 74xx-eu:DIL16
- added OUT_ROM_LOWER, OUT_ROM_UPPER: AT28C64B, ic-package:DIL28-6
- added OUT_SEGMENT_LOWER, OUT_SEGMENT_UPPER: LED, special:7SEG-13
- added SELECTOR_PARAM_: 74LS139N, 74xx-eu:DIL16
- CLK_MODE, CLK_TRIGGER: value (none) -> SWITCH
- DATABUS_2, DATABUS_3, DATABUS_4, DATABUS_5, DATABUS_6, DATABUS_7, DATABUS_8, FLAG_1, FLAG_2, FLAG_3, FLAG_4, FLAG_5, FLAG_6, FLAG_7, FLAG_8, LED_A_REG_1, LED_A_REG_2, LED_A_REG_3, LED_A_REG_4, LED_A_REG_5, LED_A_REG_6, LED_A_REG_7, LED_A_REG_8, LED_B_REG_1, LED_B_REG_2, LED_B_REG_3, LED_B_REG_4, LED_B_REG_5, LED_B_REG_6, LED_B_REG_7, LED_B_REG_8, OVERFLOW_FLAG, POSITIVE_FLAG, USTEP_1, USTEP_2, USTEP_3, USTEP_4, USTEP_5: value (none) -> LED
- INVERTED_CLK_LED: value White -> LED
- ZERO_FLAG: value (none) -> 220
- renumbered ADDR_REG_A_LOWER to REG_A_LOWER, ADDR_REG_A_UPPER to REG_A_UPPER, ADDR_REG_CALC_LOWER to REG_CALC_LOWER, ADDR_REG_CALC_UPPER to REG_CALC_UPPER, ADDR_REG_PARAM_LOWER to REG_PARAM_LOWER, ADDR_REG_PARAM_UPPER to REG_PARAM_UPPER, BRANCH_SELECTOR to SELECTOR_BRANCH_, IC1 to KEYBOARD_SHIFT_UPPER, IC2 to KEYBOARD_SHIFT_LOWER, IC4 to NOR_GATE_, INSRUCTION_REGISTER_SELECTOR_LOWER to SELECTOR_INSRUCTION_LOWER, INSRUCTION_REGISTER_SELECTOR_UPPER to SELECTOR_INSRUCTION_UPPER, INSTRUCTION_MEMORY_3 to KEYBOARD_ASCII_TABLE, NOT_GATE1 to NOT_GATE1_, SELECTOR_RAM_ to SELECTOR_STACK_
Connections:
- net N$10 renamed CTRL_SIG_19_(STACK_POP)
- net N$5 renamed RAW_INP_MODE
- removed net 1_PLACE: ADDR_MEM_REG_LOWER.11, DATABUS_1.A, EXTENSION.1, INSTRUC_REGISTER_LOWER.11, KEYBOARD_ASCII_TABLE.11, MICRO_COUNTER_LOWER.3, OUTPUT_BUFFER_ALU.2, OUTPUT_BUFFER_CALC_REG.11, OUTPUT_BUFFER_FLAGS.2, OUTPUT_BUFFER_INSTRUCTION.11, OUTPUT_BUFFER_MEMORY.11, OUTPUT_BUFFER_PARAM_REG.11, OUTPUT_BUFFER_PC.11, OUTPUT_BUFFER_RAM.18, OUTPUT_BUFFER_REG_A.11, PROGRAM_COUNTER_LOWER.3, RAM_ADDR_LOWER.14, REG_A_LOWER.11, REG_CALC_LOWER.11, REG_PARAM_LOWER.11, XOR_GATE_1.2
- new net 1_PLACE1: ADDR_MEM_REG_LOWER.11, DATABUS_1.A, EXTENSION.1, FIFO_STACK.6, FIFO_STACK.9, INSTRUC_REGISTER_LOWER.11, MICRO_COUNTER_LOWER.3, OUTPUT_BUFFER_ALU.2, OUTPUT_BUFFER_CALC_REG.11, OUTPUT_BUFFER_FLAGS.2, OUTPUT_BUFFER_INSTRUCTION.11, OUTPUT_BUFFER_KEYBOARD.2, OUTPUT_BUFFER_MEMORY.11, OUTPUT_BUFFER_PARAM_REG.11, OUTPUT_BUFFER_PC.11, OUTPUT_BUFFER_RAM.18, OUTPUT_BUFFER_REG_A.11, OUT_REG_LOWER.11, PROGRAM_COUNTER_LOWER.3, RAM_ADDR_LOWER.14, REG_A_LOWER.11, REG_CALC_LOWER.11, REG_PARAM_LOWER.11, XOR_GATE_1.2
- new net CTRL_SIG_18_(STACK_PUSH): INSTRUCTION_MEMORY_2.12, SELECTOR_PARAM_.14, SELECTOR_STACK_.13
- new net CTRL_SIG_20_(OUT_REG): INSTRUCTION_MEMORY_2.15, OUT_REG_LOWER.10, OUT_REG_LOWER.9, OUT_REG_UPPER.10, OUT_REG_UPPER.9
- new net CTRL_SIG_21_(PARAM_IN): INSTRUCTION_MEMORY_2.16, SELECTOR_PARAM_.3
- new net CTRL_SIG_22_(PARAM_OUT): INSTRUCTION_MEMORY_2.17, SELECTOR_PARAM_.2
- new net N$10: OUTPUT_BUFFER_KEYBOARD.19, SELECTOR_PARAM_.9
- new net N$101: KEYBOARD_ASCII_TABLE.19, OUTPUT_BUFFER_KEYBOARD.11
- new net N$102: KEYBOARD_ASCII_TABLE.16, OUTPUT_BUFFER_KEYBOARD.14
- new net N$103: KEYBOARD_ASCII_TABLE.18, OUTPUT_BUFFER_KEYBOARD.12
- new net N$104: KEYBOARD_ASCII_TABLE.11, OUTPUT_BUFFER_KEYBOARD.18
- new net N$105: KEYBOARD_ASCII_TABLE.13, OUTPUT_BUFFER_KEYBOARD.16
- new net N$110: KEYBOARD_ASCII_TABLE.12, OUTPUT_BUFFER_KEYBOARD.17
- new net N$128: KEYBOARD_ASCII_TABLE.15, OUTPUT_BUFFER_KEYBOARD.15
- new net N$129: OUT_ROM_UPPER.11, OUT_SEGMENT_UPPER.4
- new net N$130: OUT_ROM_UPPER.12, OUT_SEGMENT_UPPER.2
- new net N$139: OUT_ROM_UPPER.13, OUT_SEGMENT_UPPER.1
- new net N$141: OUT_REG_UPPER.3, OUT_ROM_UPPER.7
- new net N$142: OUT_REG_UPPER.4, OUT_ROM_UPPER.8
- new net N$143: OUT_REG_UPPER.5, OUT_ROM_UPPER.9
- new net N$144: OUT_REG_UPPER.6, OUT_ROM_UPPER.10
- new net N$145: OUT_REG_LOWER.6, OUT_ROM_LOWER.10
- new net N$146: OUT_REG_LOWER.5, OUT_ROM_LOWER.9
- new net N$147: OUT_REG_LOWER.4, OUT_ROM_LOWER.8
- new net N$148: OUT_REG_LOWER.3, OUT_ROM_LOWER.7
- new net N$165: OUT_ROM_LOWER.13, OUT_SEGMENT_LOWER.4
- new net N$166: OUT_ROM_LOWER.12, OUT_SEGMENT_LOWER.2
- new net N$167: OUT_ROM_LOWER.11, OUT_SEGMENT_LOWER.1
- new net N$168: OUT_ROM_LOWER.15, OUT_SEGMENT_LOWER.6
- new net N$190: OUT_ROM_LOWER.16, OUT_SEGMENT_LOWER.7
- new net N$192: OUT_ROM_LOWER.17, OUT_SEGMENT_LOWER.9
- new net N$193: OUT_ROM_LOWER.18, OUT_SEGMENT_LOWER.10
- new net N$197: OUT_ROM_LOWER.19, OUT_SEGMENT_LOWER.5
- new net N$198: OUT_ROM_UPPER.16, OUT_SEGMENT_UPPER.7
- new net N$199: OUT_ROM_UPPER.15, OUT_SEGMENT_UPPER.6
- new net N$200: OUT_ROM_UPPER.19, OUT_SEGMENT_UPPER.9
- new net N$201: OUT_ROM_UPPER.18, OUT_SEGMENT_UPPER.10
- new net N$208: OUT_ROM_UPPER.17, OUT_SEGMENT_UPPER.5
- new net N$5: INSTRUCTION_MEMORY_2.11, SELECTOR_PARAM_.13
- net 128_PLACE: now also FIFO_STACK.19, FIFO_STACK.24, OUTPUT_BUFFER_KEYBOARD.9, OUT_REG_UPPER.14; no longer KEYBOARD_ASCII_TABLE.19
- net 16_PLACE: now also FIFO_STACK.16, FIFO_STACK.27, OUTPUT_BUFFER_KEYBOARD.6, OUT_REG_UPPER.11; no longer KEYBOARD_ASCII_TABLE.16
- net 2_PLACE: now also FIFO_STACK.10, FIFO_STACK.5, OUTPUT_BUFFER_KEYBOARD.3, OUT_REG_LOWER.12; no longer KEYBOARD_ASCII_TABLE.12
- net 32_PLACE: now also FIFO_STACK.17, FIFO_STACK.26, OUTPUT_BUFFER_KEYBOARD.7, OUT_REG_UPPER.12; no longer KEYBOARD_ASCII_TABLE.17
- net 4_PLACE: now also FIFO_STACK.11, FIFO_STACK.4, OUTPUT_BUFFER_KEYBOARD.4, OUT_REG_LOWER.13; no longer KEYBOARD_ASCII_TABLE.13
- net 64_PLACE: now also FIFO_STACK.18, FIFO_STACK.25, OUTPUT_BUFFER_KEYBOARD.8, OUT_REG_UPPER.13; no longer KEYBOARD_ASCII_TABLE.18
- net 8_PLACE: now also FIFO_STACK.12, FIFO_STACK.3, OUTPUT_BUFFER_KEYBOARD.5, OUT_REG_LOWER.14; no longer KEYBOARD_ASCII_TABLE.15
- net CLOCK: now also OUT_REG_LOWER.7, OUT_REG_UPPER.7
- net CLR_REG: now also OUT_REG_LOWER.15, OUT_REG_UPPER.15
- net COUNTERS_CLEAR: now also AND_GATE3_.10; no longer AND_GATE4_.10
- net CTRL_SIG_17_(FLAG_OUT): now also SELECTOR_PARAM_.10; no longer INSTRUCTION_MEMORY_2.11
- net CTRL_SIG_21_(P_REG_IN): now also SELECTOR_PARAM_.6; no longer INP_SELECTOR.6
- net CTRL_SIG_22_(P_REG_OUT): now also SELECTOR_PARAM_.5; no longer INP_SELECTOR.5
- net END_CRNT_CMD: now also AND_GATE3_.9; no longer AND_GATE4_.9
- net END_CRNT_CMD&&BTN_PRESS: now also AND_GATE3_.8; no longer AND_GATE4_.8
- net GND: now also FIFO_STACK.14, FIFO_STACK.2, FIFO_STACK.7, KEYBOARD_ASCII_TABLE.20, KEYBOARD_ASCII_TABLE.21, KEYBOARD_ASCII_TABLE.22, KEYBOARD_ASCII_TABLE.23, KEYBOARD_ASCII_TABLE.24, KEYBOARD_ASCII_TABLE.25, OUTPUT_BUFFER_KEYBOARD.1, OUTPUT_BUFFER_KEYBOARD.10, OUT_REG_LOWER.1, OUT_REG_LOWER.2, OUT_REG_LOWER.8, OUT_REG_UPPER.1, OUT_REG_UPPER.2, OUT_REG_UPPER.8, OUT_ROM_LOWER.14, OUT_ROM_LOWER.2, OUT_ROM_LOWER.20, OUT_ROM_LOWER.21, OUT_ROM_LOWER.22, OUT_ROM_LOWER.23, OUT_ROM_LOWER.24, OUT_ROM_LOWER.25, OUT_ROM_LOWER.3, OUT_ROM_LOWER.4, OUT_ROM_LOWER.5, OUT_ROM_LOWER.6, OUT_ROM_UPPER.14, OUT_ROM_UPPER.2, OUT_ROM_UPPER.20, OUT_ROM_UPPER.21, OUT_ROM_UPPER.22, OUT_ROM_UPPER.23, OUT_ROM_UPPER.24, OUT_ROM_UPPER.25, OUT_ROM_UPPER.3, OUT_ROM_UPPER.4, OUT_ROM_UPPER.5, OUT_ROM_UPPER.6, OUT_SEGMENT_LOWER.3, OUT_SEGMENT_LOWER.8, OUT_SEGMENT_UPPER.3, OUT_SEGMENT_UPPER.8, SELECTOR_PARAM_.1, SELECTOR_PARAM_.15, SELECTOR_PARAM_.8; no longer IC5.7, INP_SELECTOR.1, INP_SELECTOR.8
- net INPUT_CTRL: now also SELECTOR_PARAM_.7, XOR_GATE_2.13; no longer IC5.2, INP_SELECTOR.7, KEYBOARD_ASCII_TABLE.22
- net N$107: now also AND_GATE3_.1; no longer AND_GATE3_.9
- net N$113: now also XOR_GATE_2.12; no longer IC5.1
- net N$127: now also XOR_GATE_2.11; no longer IC5.3
- net N$226: now also AND_GATE3_.2, NOT_GATE_.8; no longer AND_GATE3_.10, NOT_GATE_.10
- net N$26: now also KEYBOARD_ASCII_TABLE.17, OUTPUT_BUFFER_KEYBOARD.13; no longer INSTRUCTION_MEMORY_2.12, SELECTOR_STACK_.13
- net N$40: now also FIFO_STACK.1, SELECTOR_STACK_.10; no longer INP_SELECTOR.3, INSTRUCTION_MEMORY_2.16
- net N$56: now also FIFO_STACK.15, SELECTOR_STACK_.11; no longer INP_SELECTOR.2, INSTRUCTION_MEMORY_2.17
- net PC_LOAD: now also AND_GATE3_.3; no longer AND_GATE3_.8
- net PC_LOAD_SIGNAL: now also NOT_GATE_.9; no longer NOT_GATE_.11
- net VCC: now also FIFO_STACK.28, OUTPUT_BUFFER_KEYBOARD.20, OUT_REG_LOWER.16, OUT_REG_UPPER.16, OUT_ROM_LOWER.27, OUT_ROM_LOWER.28, OUT_ROM_UPPER.27, OUT_ROM_UPPER.28, SELECTOR_PARAM_.16; no longer IC5.14, INP_SELECTOR.16

Commit message: update
Connections:
- new net N$10: SELECTOR_INSRUCTION_LOWER.9, SELECTOR_PARAM_.14
- net CTRL_SIG_17_(FLAG_OUT): now also INSTRUCTION_MEMORY_2.11; no longer SELECTOR_PARAM_.10
- net CTRL_SIG_18_(STACK_PUSH): no longer SELECTOR_PARAM_.14
- net MEMORY_IN: now also SELECTOR_PARAM_.10; no longer SELECTOR_INSRUCTION_LOWER.12
- net MEMORY_OUT: now also SELECTOR_PARAM_.11; no longer SELECTOR_INSRUCTION_LOWER.9
- net N$5: now also SELECTOR_INSRUCTION_LOWER.12; no longer INSTRUCTION_MEMORY_2.11
Changed lines of the file:
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@@
 <signal name="MEMORY_OUT">
 <contactref element="NOT_GATE1_" pad="9"/>
-<contactref element="SELECTOR_INSRUCTION_LOWER" pad="9"/>
-<wire x1="133.35" y1="228.6" x2="54.61" y2="113.03" width="0" layer="19" extent="1-1"/>
+<contactref element="SELECTOR_PARAM_" pad="11"/>
+<wire x1="133.35" y1="228.6" x2="15.24" y2="-139.7" width="0" layer="19" extent="1-1"/>
 </signal>
 <signal name="~MEMORY_OUT">
@@
 </signal>
 <signal name="MEMORY_IN">
-<contactref element="SELECTOR_INSRUCTION_LOWER" pad="12"/>
 <contactref element="NOT_GATE1_" pad="5"/>
-<wire x1="125.73" y1="231.14" x2="46.99" y2="113.03" width="0" layer="19" extent="1-1"/>
+<contactref element="SELECTOR_PARAM_" pad="10"/>
+<wire x1="125.73" y1="231.14" x2="17.78" y2="-139.7" width="0" layer="19" extent="1-1"/>
 </signal>
 <signal name="16_PLACE" class="1">
@@
 <signal name="CTRL_SIG_17_(FLAG_OUT)">
 <contactref element="NOT_GATE_" pad="1"/>
-<contactref element="SELECTOR_PARAM_" pad="10"/>
-<wire x1="17.78" y1="-139.7" x2="125.73" y2="262.89" width="0" layer="19" extent="1-1"/>
+<contactref element="INSTRUCTION_MEMORY_2" pad="11"/>
+<wire x1="125.73" y1="262.89" x2="27.94" y2="170.18" width="0" layer="19" extent="1-1"/>
 </signal>
 <signal name="REG_P_128PLACE">
@@
 <contactref element="INSTRUCTION_MEMORY_2" pad="12"/>
 <contactref element="SELECTOR_STACK_" pad="13"/>
-<contactref element="SELECTOR_PARAM_" pad="14"/>
 <wire x1="77.47" y1="54.61" x2="27.94" y2="167.64" width="0" layer="19" extent="1-1"/>
-<wire x1="7.62" y1="-139.7" x2="77.47" y2="54.61" width="0" layer="19" extent="1-1"/>
 </signal>
 <signal name="RAW_INP_MODE">
@@
 <contactref element="FIFO_STACK" pad="15"/>
 <wire x1="35.56" y1="-128.27" x2="77.47" y2="49.53" width="0" layer="19" extent="1-1"/>
-</signal>
-<signal name="N$5">
-<contactref element="INSTRUCTION_MEMORY_2" pad="11"/>
-<contactref element="SELECTOR_PARAM_" pad="13"/>
-<wire x1="10.16" y1="-139.7" x2="27.94" y2="170.18" width="0" layer="19" extent="1-1"/>
-</signal>
-<signal name="N$10">
-<contactref element="SELECTOR_PARAM_" pad="9"/>
-<contactref element="OUTPUT_BUFFER_KEYBOARD" pad="19"/>
-<wire x1="20.32" y1="-139.7" x2="5.08" y2="-151.13" width="0" layer="19" extent="1-1"/>
 </signal>
 <signal name="N$26" class="1">
@@
 <wire x1="30.48" y1="-232.41" x2="-2.54" y2="-245.11" width="0" layer="19" extent="1-1"/>
 </signal>
+<signal name="N$5">
+<contactref element="SELECTOR_PARAM_" pad="13"/>
+<contactref element="SELECTOR_INSRUCTION_LOWER" pad="12"/>
+<wire x1="10.16" y1="-139.7" x2="46.99" y2="113.03" width="0" layer="19" extent="1-1"/>
+</signal>
+<signal name="N$10">
+<contactref element="SELECTOR_INSRUCTION_LOWER" pad="9"/>
+<contactref element="SELECTOR_PARAM_" pad="14"/>
+<wire x1="7.62" y1="-139.7" x2="54.61" y2="113.03" width="0" layer="19" extent="1-1"/>
+</signal>
+<signal name="N$210">
+<contactref element="OUTPUT_BUFFER_KEYBOARD" pad="19"/>
+<contactref element="SELECTOR_PARAM_" pad="9"/>
+<wire x1="20.32" y1="-139.7" x2="5.08" y2="-151.13" width="0" layer="19" extent="1-1"/>
+</signal>
 </signals>

Commit message: update
Parts:
- removed FIFO_STACK: 71256SA15TPG, ic-package:DIL28-3
- added IC1: 4161N, 40xx:DIL16
- added RAM1: 71256SA15TPG, ic-package:DIL28-3
Connections:
- removed net N$40: FIFO_STACK.1, SELECTOR_STACK_.10
- removed net N$56: FIFO_STACK.15, SELECTOR_STACK_.11
- new net STACK_POP: SELECTOR_STACK_.11
- new net STACK_PUSH: SELECTOR_STACK_.10
- new net VDD: IC1.16
- new net VSS: IC1.8
- net 128_PLACE: no longer FIFO_STACK.19, FIFO_STACK.24
- net 16_PLACE: no longer FIFO_STACK.16, FIFO_STACK.27
- net 1_PLACE1: no longer FIFO_STACK.6, FIFO_STACK.9
- net 2_PLACE: no longer FIFO_STACK.10, FIFO_STACK.5
- net 32_PLACE: no longer FIFO_STACK.17, FIFO_STACK.26
- net 4_PLACE: no longer FIFO_STACK.11, FIFO_STACK.4
- net 64_PLACE: no longer FIFO_STACK.18, FIFO_STACK.25
- net 8_PLACE: no longer FIFO_STACK.12, FIFO_STACK.3
- net GND: no longer FIFO_STACK.14, FIFO_STACK.2, FIFO_STACK.7
- net VCC: no longer FIFO_STACK.28
