File: V4/Full.sch (EAGLE design)
At the start: 206 parts, among them X1 SSW-103-02-G-S

Commit message: update
Parts:
- added INP_SELECTOR: 74AC139N, 74xx-eu:74AC139N
Connections:
- new net N$40: INP_SELECTORA.B, INSTRUCTION_MEMORY_2.16
- new net N$56: INP_SELECTORA.A, INSTRUCTION_MEMORY_2.17
- net CTRL_SIG_21_(P_REG_IN): now also INP_SELECTORA.Y2; no longer INSTRUCTION_MEMORY_2.16
- net CTRL_SIG_22_(P_REG_OUT): now also INP_SELECTORA.Y1; no longer INSTRUCTION_MEMORY_2.17
- net GND: now also INP_SELECTORA.G
Changed lines of the file:
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@@
 <part name="SELECTOR_RAM_" library="74xx-eu" library_urn="urn:adsk.eagle:library:85" deviceset="74*139" device="N" package3d_urn="urn:adsk.eagle:package:922/2" technology="LS"/>
 <part name="GND45" library="supply1" library_urn="urn:adsk.eagle:library:371" deviceset="GND" device=""/>
+<part name="INP_SELECTOR" library="74xx-eu" library_urn="urn:adsk.eagle:library:85" deviceset="74*139" device="N" package3d_urn="urn:adsk.eagle:package:922/2" technology="AC"/>
+<part name="GND57" library="supply1" library_urn="urn:adsk.eagle:library:371" deviceset="GND" device=""/>
 </parts>
 <sheets>
@@
 <text x="-45.72" y="76.2" size="1.778" layer="91" rot="R270">CLOCK</text>
 <text x="-119.38" y="-172.72" size="1.778" layer="91">Flag Out</text>
-<text x="-99.06" y="-162.56" size="1.778" layer="91">Parameter Register IN</text>
-<text x="-99.06" y="-160.02" size="1.778" layer="91">Parameter Register OUT</text>
+<text x="-147.32" y="-162.56" size="1.778" layer="91">Parameter Register IN</text>
+<text x="-147.32" y="-160.02" size="1.778" layer="91">Parameter Register OUT</text>
 <text x="289.56" y="-12.7" size="1.778" layer="91">OF</text>
 <text x="276.86" y="-25.4" size="1.778" layer="91">PF</text>
@@
 </instance>
 <instance part="GND45" gate="1" x="-167.64" y="-187.96" smashed="yes" rot="R270"/>
+<instance part="INP_SELECTOR" gate="A" x="-88.9" y="-160.02" smashed="yes">
+<attribute name="NAME" x="-96.52" y="-154.305" size="1.778" layer="95"/>
+<attribute name="VALUE" x="-96.52" y="-170.18" size="1.778" layer="96"/>
+</instance>
+<instance part="GND57" gate="1" x="-104.14" y="-165.1" smashed="yes" rot="R270"/>
 </instances>
 <busses>
@@
 <pinref part="GND45" gate="1" pin="GND"/>
 </segment>
+<segment>
+<pinref part="INP_SELECTOR" gate="A" pin="G"/>
+<pinref part="GND57" gate="1" pin="GND"/>
+</segment>
 </net>
 <net name="N$1" class="0">
@@
 <net name="CTRL_SIG_21_(P_REG_IN)" class="0">
 <segment>
-<pinref part="INSTRUCTION_MEMORY_2" gate="G$1" pin="16"/>
-<wire x1="-147.32" y1="-162.56" x2="-68.58" y2="-162.56" width="0.1524" layer="91"/>
 <wire x1="-68.58" y1="-162.56" x2="-68.58" y2="-152.4" width="0.1524" layer="91"/>
 <wire x1="-68.58" y1="-152.4" x2="-50.8" y2="-152.4" width="0.1524" layer="91"/>
@@
 <wire x1="243.84" y1="-170.18" x2="243.84" y2="-177.8" width="0.1524" layer="91"/>
 <pinref part="NOT_GATE2_" gate="B" pin="I"/>
+<pinref part="INP_SELECTOR" gate="A" pin="Y2"/>
+<wire x1="-68.58" y1="-162.56" x2="-76.2" y2="-162.56" width="0.1524" layer="91"/>
 </segment>
 </net>
 <net name="CTRL_SIG_22_(P_REG_OUT)" class="0">
 <segment>
-<pinref part="INSTRUCTION_MEMORY_2" gate="G$1" pin="17"/>
-<wire x1="-147.32" y1="-160.02" x2="-71.12" y2="-160.02" width="0.1524" layer="91"/>
 <wire x1="-71.12" y1="-160.02" x2="-71.12" y2="-154.94" width="0.1524" layer="91"/>
 <wire x1="-71.12" y1="-154.94" x2="-48.26" y2="-154.94" width="0.1524" layer="91"/>
@@
 <wire x1="144.78" y1="-195.58" x2="144.78" y2="-132.08" width="0.1524" layer="91"/>
 <pinref part="NOT_GATE2_" gate="A" pin="I"/>
+<pinref part="INP_SELECTOR" gate="A" pin="Y1"/>
+<wire x1="-76.2" y1="-160.02" x2="-71.12" y2="-160.02" width="0.1524" layer="91"/>
 </segment>
 </net>
@@
 </segment>
 </net>
+<net name="N$40" class="0">
+<segment>
+<pinref part="INP_SELECTOR" gate="A" pin="B"/>
+<pinref part="INSTRUCTION_MEMORY_2" gate="G$1" pin="16"/>
+<wire x1="-101.6" y1="-160.02" x2="-101.6" y2="-162.56" width="0.1524" layer="91"/>
+<wire x1="-101.6" y1="-162.56" x2="-147.32" y2="-162.56" width="0.1524" layer="91"/>
+</segment>
+</net>
+<net name="N$56" class="0">
+<segment>
+<pinref part="INSTRUCTION_MEMORY_2" gate="G$1" pin="17"/>
+<wire x1="-147.32" y1="-160.02" x2="-104.14" y2="-160.02" width="0.1524" layer="91"/>
+<wire x1="-104.14" y1="-160.02" x2="-104.14" y2="-157.48" width="0.1524" layer="91"/>
+<pinref part="INP_SELECTOR" gate="A" pin="A"/>
+<wire x1="-104.14" y1="-157.48" x2="-101.6" y2="-157.48" width="0.1524" layer="91"/>
+</segment>
+</net>
