File: V4/Full.sch (EAGLE design)
At the start: 212 parts, among them IC1 74LS595N, IC2 74LS595N, X1 SSW-103-02-G-S

Commit message: update
Parts:
- removed IC4: (no value), ic-package:DIL28
- added INSTRUCTION_MEMORY_3: AT28C64B, ic-package:DIL28
Connections:
- removed net N$84: IC4.10
- removed net N$96: IC2A.QA, IC4.19
- removed net N$99: IC1A.QG, IC4.17
- new net N$101: IC1A.QG, INSTRUCTION_MEMORY_3.17
- new net N$113: IC2A.QA, INSTRUCTION_MEMORY_3.19
- net GND: now also IC1A.SCL, IC2A.SCL, INSTRUCTION_MEMORY_3.14, INSTRUCTION_MEMORY_3.2; no longer IC4.14
- net N$102: now also INSTRUCTION_MEMORY_3.3; no longer IC4.3
- net N$103: now also INSTRUCTION_MEMORY_3.4; no longer IC4.4
- net N$104: now also INSTRUCTION_MEMORY_3.5; no longer IC4.5
- net N$105: now also INSTRUCTION_MEMORY_3.6; no longer IC4.6
- net N$106: now also INSTRUCTION_MEMORY_3.7; no longer IC4.7
- net N$108: now also INSTRUCTION_MEMORY_3.8; no longer IC4.8
- net N$109: now also INSTRUCTION_MEMORY_3.9; no longer IC4.9
- net N$80: now also INSTRUCTION_MEMORY_3.11; no longer IC4.11
- net N$81: now also INSTRUCTION_MEMORY_3.12; no longer IC4.12
- net N$82: now also INSTRUCTION_MEMORY_3.13; no longer IC4.13
- net N$85: now also INSTRUCTION_MEMORY_3.16; no longer IC4.16
- net N$86: now also INSTRUCTION_MEMORY_3.10; no longer IC1A.SCL, IC2A.SCL
- net N$95: now also INSTRUCTION_MEMORY_3.18; no longer IC4.18
- net N$98: now also INSTRUCTION_MEMORY_3.15; no longer IC4.15
- net VCC: now also INSTRUCTION_MEMORY_3.27, INSTRUCTION_MEMORY_3.28; no longer IC4.27, IC4.28

Commit message: update
Parts:
- added OUTPUT_BUFFER_ALU1: 74LS245N, 74xx-eu:74LS245N
Connections:
- net N$61 renamed INPUT_CTRL
- removed net N$101: IC1A.QG, INSTRUCTION_MEMORY_3.17
- removed net N$102: INSTRUCTION_MEMORY_3.3
- removed net N$103: INSTRUCTION_MEMORY_3.4
- removed net N$104: INSTRUCTION_MEMORY_3.5
- removed net N$105: INSTRUCTION_MEMORY_3.6
- removed net N$106: INSTRUCTION_MEMORY_3.7
- removed net N$108: INSTRUCTION_MEMORY_3.8
- removed net N$109: INSTRUCTION_MEMORY_3.9
- removed net N$113: IC2A.QA, INSTRUCTION_MEMORY_3.19
- removed net N$80: IC1A.QB, INSTRUCTION_MEMORY_3.11
- removed net N$81: IC1A.QC, INSTRUCTION_MEMORY_3.12
- removed net N$82: IC1A.QD, INSTRUCTION_MEMORY_3.13
- removed net N$85: IC1A.QF, INSTRUCTION_MEMORY_3.16
- removed net N$86: INSTRUCTION_MEMORY_3.10
- removed net N$95: IC1A.QH, INSTRUCTION_MEMORY_3.18
- removed net N$98: IC1A.QE, INSTRUCTION_MEMORY_3.15
- new net N$61: IC1A.G, IC2A.G
- net GND: no longer IC1A.G, IC2A.G
Other:
- note added: "RAM"
- moved on the sheet: IC1, IC2, INSTRUCTION_MEMORY_3, KEYBOARD-1
