File: V4/Full.sch (EAGLE design)
At the start: 216 parts, among them IC1 74LS595N, IC2 74LS595N, IC4 74LS02N, IC5 74S86N, X1 SSW-103-02-G-S

Commit message: update
Parts:
- added D1: 1N4728, diode:1N4728
Connections:
- net N$106: now also D1.C
- net N$63: now also D1.A
Other:
- note removed: "DIODE"
Changed lines of the file:
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@@
 <layer number="97" name="Info" color="7" fill="1" visible="yes" active="yes"/>
 <layer number="98" name="Guide" color="6" fill="1" visible="yes" active="yes"/>
+<layer number="99" name="SpiceOrder" color="5" fill="1" visible="yes" active="yes"/>
 </layers>
 <schematic xreflabel="%F%N/%S.%C%R" xrefpart="/%S.%C%R">
@@
 <part name="IC4" library="74xx-eu" library_urn="urn:adsk.eagle:library:85" deviceset="74*02" device="N" package3d_urn="urn:adsk.eagle:package:16407/2" technology="LS"/>
 <part name="IC5" library="74xx-eu" library_urn="urn:adsk.eagle:library:85" deviceset="74*86" device="N" package3d_urn="urn:adsk.eagle:package:16407/2" technology="S"/>
+<part name="D1" library="diode" library_urn="urn:adsk.eagle:library:210" deviceset="1N4728" device="" package3d_urn="urn:adsk.eagle:package:43341/1"/>
 </parts>
 <sheets>
@@
 <text x="309.88" y="172.72" size="1.778" layer="91">Data</text>
 <text x="-17.78" y="-180.34" size="1.778" layer="91">RAM</text>
-<text x="297.18" y="109.22" size="1.778" layer="91" rot="R90">DIODE</text>
 </plain>
 <instances>
@@
 <instance part="P+25" gate="VCC" x="304.8" y="127" smashed="yes" rot="R90"/>
 <instance part="GND62" gate="1" x="309.88" y="147.32" smashed="yes" rot="R180"/>
-<instance part="R6" gate="G$1" x="302.26" y="114.3" smashed="yes" rot="R270">
-<attribute name="VALUE" x="298.958" y="118.11" size="1.778" layer="96" rot="R270"/>
-</instance>
+<instance part="R6" gate="G$1" x="302.26" y="114.3" smashed="yes" rot="R270"/>
 <instance part="C4" gate="G$1" x="304.8" y="104.14" smashed="yes" rot="R90"/>
 <instance part="NOT_GATE3_" gate="D" x="256.54" y="91.44" smashed="yes" rot="R180"/>
@@
 <instance part="NOT_GATE_" gate="B" x="302.26" y="91.44" smashed="yes" rot="R180"/>
 <instance part="NOT_GATE_" gate="C" x="195.58" y="91.44" smashed="yes" rot="R180"/>
+<instance part="D1" gate="1" x="297.18" y="116.84" smashed="yes" rot="R270"/>
 </instances>
 <busses>
@@
 <wire x1="297.18" y1="119.38" x2="302.26" y2="119.38" width="0.1524" layer="91"/>
 <junction x="302.26" y="119.38"/>
+<pinref part="D1" gate="1" pin="A"/>
 </segment>
 </net>
@@
 <wire x1="302.26" y1="104.14" x2="297.18" y2="104.14" width="0.1524" layer="91"/>
 <junction x="302.26" y="104.14"/>
-<wire x1="297.18" y1="104.14" x2="297.18" y2="109.22" width="0.1524" layer="91"/>
 <wire x1="302.26" y1="104.14" x2="302.26" y2="101.6" width="0.1524" layer="91"/>
 <wire x1="180.34" y1="99.06" x2="292.1" y2="99.06" width="0.1524" layer="91"/>
@@
 <pinref part="IC4" gate="A" pin="I1"/>
 <wire x1="180.34" y1="96.52" x2="180.34" y2="99.06" width="0.1524" layer="91"/>
+<pinref part="D1" gate="1" pin="C"/>
+<wire x1="297.18" y1="104.14" x2="297.18" y2="114.3" width="0.1524" layer="91"/>
 </segment>
 </net>

Commit message: update
Parts:
- removed IC3: (no value), ic-package:DIL28
- removed IC5: 74S86N, 74xx-eu:74S86N
- removed INP_SELECTOR: 74AC139N, 74xx-eu:74AC139N
- added FIFO_STACK: 71256SA15TPG, ic-package:DIL28-3
- added OUTPUT_BUFFER_KEYBOARD: 74LS245N, 74xx-eu:74LS245N
- added OUT_REG_LOWER, OUT_REG_UPPER: 74LS173N, 74xx-eu:74LS173N
- added OUT_ROM_LOWER, OUT_ROM_UPPER: AT28C64B, ic-package:DIL28
- added OUT_SEGMENT_LOWER, OUT_SEGMENT_UPPER: LED, special:7SEG-CK
- added SELECTOR_PARAM_: 74LS139N, 74xx-eu:74LS139N
- CLK_MODE, CLK_TRIGGER: value (none) -> SWITCH
- DATABUS_2, DATABUS_3, DATABUS_4, DATABUS_5, DATABUS_6, DATABUS_7, DATABUS_8, FLAG_1, FLAG_2, FLAG_3, FLAG_4, FLAG_5, FLAG_6, FLAG_7, FLAG_8, LED_A_REG_1, LED_A_REG_2, LED_A_REG_3, LED_A_REG_4, LED_A_REG_5, LED_A_REG_6, LED_A_REG_7, LED_A_REG_8, LED_B_REG_1, LED_B_REG_2, LED_B_REG_3, LED_B_REG_4, LED_B_REG_5, LED_B_REG_6, LED_B_REG_7, LED_B_REG_8, OVERFLOW_FLAG, POSITIVE_FLAG, USTEP_1, USTEP_2, USTEP_3, USTEP_4, USTEP_5: value (none) -> LED
- INVERTED_CLK_LED: value White -> LED
- ZERO_FLAG: value (none) -> 220
- renumbered ADDR_REG_A_LOWER to REG_A_LOWER, ADDR_REG_A_UPPER to REG_A_UPPER, ADDR_REG_CALC_LOWER to REG_CALC_LOWER, ADDR_REG_CALC_UPPER to REG_CALC_UPPER, ADDR_REG_PARAM_LOWER to REG_PARAM_LOWER, ADDR_REG_PARAM_UPPER to REG_PARAM_UPPER, BRANCH_SELECTOR to SELECTOR_BRANCH_, IC1 to KEYBOARD_SHIFT_UPPER, IC2 to KEYBOARD_SHIFT_LOWER, IC4 to NOR_GATE_, INSRUCTION_REGISTER_SELECTOR_LOWER to SELECTOR_INSRUCTION_LOWER, INSRUCTION_REGISTER_SELECTOR_UPPER to SELECTOR_INSRUCTION_UPPER, INSTRUCTION_MEMORY_3 to KEYBOARD_ASCII_TABLE, NOT_GATE1 to NOT_GATE1_, SELECTOR_RAM_ to SELECTOR_STACK_
Connections:
- net N$10 renamed CTRL_SIG_19_(STACK_POP)
- net N$5 renamed RAW_INP_MODE
- removed net 1_PLACE: ADDR_MEM_REG_LOWERA.D4, DATABUS_1.A, EXTENSION-1.1, INSTRUC_REGISTER_LOWERA.D4, KEYBOARD_ASCII_TABLE.11, MICRO_COUNTER_LOWER.3, OUTPUT_BUFFER_ALUA.A1, OUTPUT_BUFFER_CALC_REGA.B8, OUTPUT_BUFFER_FLAGSA.A1, OUTPUT_BUFFER_INSTRUCTIONA.B8, OUTPUT_BUFFER_MEMORYA.B8, OUTPUT_BUFFER_PARAM_REGA.B8, OUTPUT_BUFFER_PCA.B8, OUTPUT_BUFFER_RAMA.B1, OUTPUT_BUFFER_REG_AA.B8, PROGRAM_COUNTER_LOWER.3, RAM_ADDR_LOWERA.D1, REG_A_LOWERA.D4, REG_CALC_LOWERA.D4, REG_PARAM_LOWERA.D4, XOR_GATE_1A.I1
- new net 1_PLACE1: ADDR_MEM_REG_LOWERA.D4, DATABUS_1.A, EXTENSION-1.1, FIFO_STACK.6, FIFO_STACK.9, INSTRUC_REGISTER_LOWERA.D4, MICRO_COUNTER_LOWER.3, OUTPUT_BUFFER_ALUA.A1, OUTPUT_BUFFER_CALC_REGA.B8, OUTPUT_BUFFER_FLAGSA.A1, OUTPUT_BUFFER_INSTRUCTIONA.B8, OUTPUT_BUFFER_KEYBOARDA.A1, OUTPUT_BUFFER_MEMORYA.B8, OUTPUT_BUFFER_PARAM_REGA.B8, OUTPUT_BUFFER_PCA.B8, OUTPUT_BUFFER_RAMA.B1, OUTPUT_BUFFER_REG_AA.B8, OUT_REG_LOWERA.D4, PROGRAM_COUNTER_LOWER.3, RAM_ADDR_LOWERA.D1, REG_A_LOWERA.D4, REG_CALC_LOWERA.D4, REG_PARAM_LOWERA.D4, XOR_GATE_1A.I1
- new net CTRL_SIG_18_(STACK_PUSH): INSTRUCTION_MEMORY_2.12, SELECTOR_PARAM_B.A, SELECTOR_STACK_B.B
- new net CTRL_SIG_20_(OUT_REG): INSTRUCTION_MEMORY_2.15, OUT_REG_LOWERA.G1, OUT_REG_LOWERA.G2, OUT_REG_UPPERA.G1, OUT_REG_UPPERA.G2
- new net CTRL_SIG_21_(PARAM_IN): INSTRUCTION_MEMORY_2.16, SELECTOR_PARAM_A.B
- new net CTRL_SIG_22_(PARAM_OUT): INSTRUCTION_MEMORY_2.17, SELECTOR_PARAM_A.A
- new net N$10: OUTPUT_BUFFER_KEYBOARDA.G, SELECTOR_PARAM_B.Y3
- new net N$101: KEYBOARD_ASCII_TABLE.19, OUTPUT_BUFFER_KEYBOARDA.B8
- new net N$102: KEYBOARD_ASCII_TABLE.16, OUTPUT_BUFFER_KEYBOARDA.B5
- new net N$103: KEYBOARD_ASCII_TABLE.18, OUTPUT_BUFFER_KEYBOARDA.B7
- new net N$104: KEYBOARD_ASCII_TABLE.11, OUTPUT_BUFFER_KEYBOARDA.B1
- new net N$105: KEYBOARD_ASCII_TABLE.13, OUTPUT_BUFFER_KEYBOARDA.B3
- new net N$110: KEYBOARD_ASCII_TABLE.12, OUTPUT_BUFFER_KEYBOARDA.B2
- new net N$128: KEYBOARD_ASCII_TABLE.15, OUTPUT_BUFFER_KEYBOARDA.B4
- new net N$129: OUT_ROM_UPPER.11, OUT_SEGMENT_UPPER.C
- new net N$130: OUT_ROM_UPPER.12, OUT_SEGMENT_UPPER.D
- new net N$139: OUT_ROM_UPPER.13, OUT_SEGMENT_UPPER.E
- new net N$141: OUT_REG_UPPERA.Q1, OUT_ROM_UPPER.7
- new net N$142: OUT_REG_UPPERA.Q2, OUT_ROM_UPPER.8
- new net N$143: OUT_REG_UPPERA.Q3, OUT_ROM_UPPER.9
- new net N$144: OUT_REG_UPPERA.Q4, OUT_ROM_UPPER.10
- new net N$145: OUT_REG_LOWERA.Q4, OUT_ROM_LOWER.10
- new net N$146: OUT_REG_LOWERA.Q3, OUT_ROM_LOWER.9
- new net N$147: OUT_REG_LOWERA.Q2, OUT_ROM_LOWER.8
- new net N$148: OUT_REG_LOWERA.Q1, OUT_ROM_LOWER.7
- new net N$165: OUT_ROM_LOWER.13, OUT_SEGMENT_LOWER.C
- new net N$166: OUT_ROM_LOWER.12, OUT_SEGMENT_LOWER.D
- new net N$167: OUT_ROM_LOWER.11, OUT_SEGMENT_LOWER.E
- new net N$168: OUT_ROM_LOWER.15, OUT_SEGMENT_LOWER.B
- new net N$190: OUT_ROM_LOWER.16, OUT_SEGMENT_LOWER.A
- new net N$192: OUT_ROM_LOWER.17, OUT_SEGMENT_LOWER.F
- new net N$193: OUT_ROM_LOWER.18, OUT_SEGMENT_LOWER.G
- new net N$197: OUT_ROM_LOWER.19, OUT_SEGMENT_LOWER.DP
- new net N$198: OUT_ROM_UPPER.16, OUT_SEGMENT_UPPER.A
- new net N$199: OUT_ROM_UPPER.15, OUT_SEGMENT_UPPER.B
- new net N$200: OUT_ROM_UPPER.19, OUT_SEGMENT_UPPER.F
- new net N$201: OUT_ROM_UPPER.18, OUT_SEGMENT_UPPER.G
- new net N$208: OUT_ROM_UPPER.17, OUT_SEGMENT_UPPER.DP
- new net N$5: INSTRUCTION_MEMORY_2.11, SELECTOR_PARAM_B.B
- net 128_PLACE: now also FIFO_STACK.19, FIFO_STACK.24, OUTPUT_BUFFER_KEYBOARDA.A8, OUT_REG_UPPERA.D1; no longer KEYBOARD_ASCII_TABLE.19
- net 16_PLACE: now also FIFO_STACK.16, FIFO_STACK.27, OUTPUT_BUFFER_KEYBOARDA.A5, OUT_REG_UPPERA.D4; no longer KEYBOARD_ASCII_TABLE.16
- net 2_PLACE: now also FIFO_STACK.10, FIFO_STACK.5, OUTPUT_BUFFER_KEYBOARDA.A2, OUT_REG_LOWERA.D3; no longer KEYBOARD_ASCII_TABLE.12
- net 32_PLACE: now also FIFO_STACK.17, FIFO_STACK.26, OUTPUT_BUFFER_KEYBOARDA.A6, OUT_REG_UPPERA.D3; no longer KEYBOARD_ASCII_TABLE.17
- net 4_PLACE: now also FIFO_STACK.11, FIFO_STACK.4, OUTPUT_BUFFER_KEYBOARDA.A3, OUT_REG_LOWERA.D2; no longer KEYBOARD_ASCII_TABLE.13
- net 64_PLACE: now also FIFO_STACK.18, FIFO_STACK.25, OUTPUT_BUFFER_KEYBOARDA.A7, OUT_REG_UPPERA.D2; no longer KEYBOARD_ASCII_TABLE.18
- net 8_PLACE: now also FIFO_STACK.12, FIFO_STACK.3, OUTPUT_BUFFER_KEYBOARDA.A4, OUT_REG_LOWERA.D1; no longer KEYBOARD_ASCII_TABLE.15
- net CLOCK: now also OUT_REG_LOWERA.CLK, OUT_REG_UPPERA.CLK
- net CLR_REG: now also OUT_REG_LOWERA.CLR, OUT_REG_UPPERA.CLR
- net COUNTERS_CLEAR: now also AND_GATE3_C.I1; no longer AND_GATE4_C.I1
- net CTRL_SIG_17_(FLAG_OUT): now also SELECTOR_PARAM_B.Y2; no longer INSTRUCTION_MEMORY_2.11
- net CTRL_SIG_21_(P_REG_IN): now also SELECTOR_PARAM_A.Y2; no longer INP_SELECTORA.Y2
- net CTRL_SIG_22_(P_REG_OUT): now also SELECTOR_PARAM_A.Y1; no longer INP_SELECTORA.Y1
- net END_CRNT_CMD: now also AND_GATE3_C.I0; no longer AND_GATE4_C.I0
- net END_CRNT_CMD&&BTN_PRESS: now also AND_GATE3_C.O; no longer AND_GATE4_C.O
- net GND: now also FIFO_STACK.14, FIFO_STACK.2, FIFO_STACK.7, KEYBOARD_ASCII_TABLE.20, KEYBOARD_ASCII_TABLE.21, KEYBOARD_ASCII_TABLE.22, KEYBOARD_ASCII_TABLE.23, KEYBOARD_ASCII_TABLE.24, KEYBOARD_ASCII_TABLE.25, OUTPUT_BUFFER_KEYBOARDA.DIR, OUT_REG_LOWERA.M, OUT_REG_LOWERA.N, OUT_REG_UPPERA.M, OUT_REG_UPPERA.N, OUT_ROM_LOWER.14, OUT_ROM_LOWER.2, OUT_ROM_LOWER.20, OUT_ROM_LOWER.21, OUT_ROM_LOWER.22, OUT_ROM_LOWER.23, OUT_ROM_LOWER.24, OUT_ROM_LOWER.25, OUT_ROM_LOWER.3, OUT_ROM_LOWER.4, OUT_ROM_LOWER.5, OUT_ROM_LOWER.6, OUT_ROM_UPPER.14, OUT_ROM_UPPER.2, OUT_ROM_UPPER.20, OUT_ROM_UPPER.21, OUT_ROM_UPPER.22, OUT_ROM_UPPER.23, OUT_ROM_UPPER.24, OUT_ROM_UPPER.25, OUT_ROM_UPPER.3, OUT_ROM_UPPER.4, OUT_ROM_UPPER.5, OUT_ROM_UPPER.6, OUT_SEGMENT_LOWER.CK1, OUT_SEGMENT_LOWER.CK2, OUT_SEGMENT_UPPER.CK1, OUT_SEGMENT_UPPER.CK2, SELECTOR_PARAM_A.G, SELECTOR_PARAM_B.G; no longer INP_SELECTORA.G
- net INPUT_CTRL: now also SELECTOR_PARAM_A.Y3, XOR_GATE_2D.I1; no longer IC5A.I1, INP_SELECTORA.Y3, KEYBOARD_ASCII_TABLE.22
- net N$107: now also AND_GATE3_A.I0; no longer AND_GATE3_C.I0
- net N$113: now also XOR_GATE_2D.I0; no longer IC5A.I0
- net N$127: now also XOR_GATE_2D.O; no longer IC5A.O
- net N$226: now also AND_GATE3_A.I1, NOT_GATE_D.O; no longer AND_GATE3_C.I1, NOT_GATE_E.O
- net N$26: now also KEYBOARD_ASCII_TABLE.17, OUTPUT_BUFFER_KEYBOARDA.B6; no longer INSTRUCTION_MEMORY_2.12, SELECTOR_STACK_B.B
- net N$40: now also FIFO_STACK.1, SELECTOR_STACK_B.Y2; no longer INP_SELECTORA.B, INSTRUCTION_MEMORY_2.16
- net N$56: now also FIFO_STACK.15, SELECTOR_STACK_B.Y1; no longer INP_SELECTORA.A, INSTRUCTION_MEMORY_2.17
- net PC_LOAD: now also AND_GATE3_A.O; no longer AND_GATE3_C.O
- net PC_LOAD_SIGNAL: now also NOT_GATE_D.I; no longer NOT_GATE_E.I
- net VCC: now also FIFO_STACK.28, OUT_ROM_LOWER.27, OUT_ROM_LOWER.28, OUT_ROM_UPPER.27, OUT_ROM_UPPER.28
Other:
- note added: "CLR REGISTERS"
- moved on the sheet: AUTO_CLOCK, EXTENSION-1, EXTENSION-10, EXTENSION-11, EXTENSION-2, EXTENSION-3, EXTENSION-4, EXTENSION-5, EXTENSION-6, EXTENSION-7, EXTENSION-8, EXTENSION-9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

Commit message: update
Connections:
- new net N$10: SELECTOR_INSRUCTION_LOWERA.3Y, SELECTOR_PARAM_B.A
- net CTRL_SIG_17_(FLAG_OUT): now also INSTRUCTION_MEMORY_2.11; no longer SELECTOR_PARAM_B.Y2
- net CTRL_SIG_18_(STACK_PUSH): no longer SELECTOR_PARAM_B.A
- net MEMORY_IN: now also SELECTOR_PARAM_B.Y2; no longer SELECTOR_INSRUCTION_LOWERA.4Y
- net MEMORY_OUT: now also SELECTOR_PARAM_B.Y1; no longer SELECTOR_INSRUCTION_LOWERA.3Y
- net N$5: now also SELECTOR_INSRUCTION_LOWERA.4Y; no longer INSTRUCTION_MEMORY_2.11
Changed lines of the file:
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@@
 <text x="27.94" y="45.72" size="1.778" layer="91">Reg A OUT</text>
 <text x="27.94" y="40.64" size="1.778" layer="91">Reg A IN</text>
-<text x="27.94" y="35.56" size="1.778" layer="91">Memory OUT</text>
-<text x="27.94" y="30.48" size="1.778" layer="91">Memory IN</text>
+<text x="63.5" y="33.02" size="1.778" layer="91" rot="R90">Memory OUT</text>
+<text x="66.04" y="33.02" size="1.778" layer="91" rot="R90">Memory IN</text>
 <text x="27.94" y="81.28" size="1.778" layer="91">RAM_WRITE</text>
 <text x="27.94" y="86.36" size="1.778" layer="91">RAM_ADDR_IN</text>
@@
 <instance part="SELECTOR_STACK_" gate="A" x="38.1" y="71.12" smashed="yes">
 <attribute name="NAME" x="30.48" y="76.835" size="1.778" layer="95"/>
-<attribute name="VALUE" x="30.48" y="60.96" size="1.778" layer="96"/>
 </instance>
 <instance part="SELECTOR_STACK_" gate="B" x="-132.08" y="-177.8" smashed="yes"/>
@@
 <attribute name="NAME" x="43.18" y="-118.745" size="1.778" layer="95"/>
 </instance>
-<instance part="SELECTOR_PARAM_" gate="B" x="-132.08" y="-193.04" smashed="yes"/>
-<instance part="GND88" gate="1" x="-147.32" y="-198.12" smashed="yes" rot="R270"/>
+<instance part="SELECTOR_PARAM_" gate="B" x="43.18" y="30.48" smashed="yes"/>
+<instance part="GND88" gate="1" x="30.48" y="22.86" smashed="yes"/>
 <instance part="GND89" gate="1" x="373.38" y="160.02" smashed="yes" rot="R90"/>
 <instance part="OUTPUT_BUFFER_KEYBOARD" gate="A" x="330.2" y="71.12" smashed="yes"/>
@@
 <segment>
 <pinref part="NOT_GATE1_" gate="D" pin="I"/>
-<pinref part="SELECTOR_INSRUCTION_LOWER" gate="A" pin="3Y"/>
-<wire x1="63.5" y1="127" x2="63.5" y2="35.56" width="0.1524" layer="91"/>
-<wire x1="22.86" y1="35.56" x2="63.5" y2="35.56" width="0.1524" layer="91"/>
+<wire x1="63.5" y1="127" x2="63.5" y2="30.48" width="0.1524" layer="91"/>
 <wire x1="-12.7" y1="208.28" x2="-12.7" y2="129.54" width="0.1524" layer="91"/>
 <wire x1="-12.7" y1="129.54" x2="22.86" y2="129.54" width="0.1524" layer="91"/>
 <wire x1="22.86" y1="129.54" x2="22.86" y2="127" width="0.1524" layer="91"/>
 <wire x1="22.86" y1="127" x2="63.5" y2="127" width="0.1524" layer="91"/>
+<pinref part="SELECTOR_PARAM_" gate="B" pin="Y1"/>
+<wire x1="55.88" y1="30.48" x2="63.5" y2="30.48" width="0.1524" layer="91"/>
 </segment>
 </net>
@@
 <segment>
 <wire x1="-10.16" y1="340.36" x2="66.04" y2="340.36" width="0.1524" layer="91"/>
-<wire x1="66.04" y1="340.36" x2="66.04" y2="30.48" width="0.1524" layer="91"/>
-<pinref part="SELECTOR_INSRUCTION_LOWER" gate="A" pin="4Y"/>
-<wire x1="22.86" y1="30.48" x2="66.04" y2="30.48" width="0.1524" layer="91"/>
+<wire x1="66.04" y1="340.36" x2="66.04" y2="27.94" width="0.1524" layer="91"/>
 <wire x1="-10.16" y1="340.36" x2="-10.16" y2="350.52" width="0.1524" layer="91"/>
 <pinref part="NOT_GATE1_" gate="C" pin="I"/>
 <wire x1="-10.16" y1="350.52" x2="-17.78" y2="350.52" width="0.1524" layer="91"/>
+<pinref part="SELECTOR_PARAM_" gate="B" pin="Y2"/>
+<wire x1="55.88" y1="27.94" x2="66.04" y2="27.94" width="0.1524" layer="91"/>
 </segment>
 </net>
@@
 <net name="CTRL_SIG_17_(FLAG_OUT)" class="0">
 <segment>
-<wire x1="-114.3" y1="-170.18" x2="-58.42" y2="-170.18" width="0.1524" layer="91"/>
 <wire x1="-58.42" y1="-170.18" x2="-58.42" y2="-142.24" width="0.1524" layer="91"/>
 <wire x1="-58.42" y1="-142.24" x2="-7.62" y2="-142.24" width="0.1524" layer="91"/>
 <wire x1="-7.62" y1="-142.24" x2="-7.62" y2="-45.72" width="0.1524" layer="91"/>
 <pinref part="NOT_GATE_" gate="A" pin="I"/>
-<pinref part="SELECTOR_PARAM_" gate="B" pin="Y2"/>
-<wire x1="-119.38" y1="-195.58" x2="-114.3" y2="-195.58" width="0.1524" layer="91"/>
-<wire x1="-114.3" y1="-195.58" x2="-114.3" y2="-170.18" width="0.1524" layer="91"/>
 <wire x1="-7.62" y1="-45.72" x2="109.22" y2="-45.72" width="0.1524" layer="91"/>
 <wire x1="119.38" y1="-38.1" x2="109.22" y2="-38.1" width="0.1524" layer="91"/>
 <wire x1="109.22" y1="-38.1" x2="109.22" y2="-45.72" width="0.1524" layer="91"/>
+<wire x1="-170.18" y1="-157.48" x2="-170.18" y2="-170.18" width="0.1524" layer="91"/>
+<pinref part="INSTRUCTION_MEMORY_2" gate="G$1" pin="11"/>
+<wire x1="-162.56" y1="-157.48" x2="-170.18" y2="-157.48" width="0.1524" layer="91"/>
+<wire x1="-58.42" y1="-170.18" x2="-170.18" y2="-170.18" width="0.1524" layer="91"/>
 </segment>
 </net>
@@
 <wire x1="-162.56" y1="-160.02" x2="-167.64" y2="-160.02" width="0.1524" layer="91"/>
 <pinref part="SELECTOR_STACK_" gate="B" pin="B"/>
-<wire x1="-144.78" y1="-177.8" x2="-149.86" y2="-177.8" width="0.1524" layer="91"/>
-<wire x1="-149.86" y1="-177.8" x2="-167.64" y2="-177.8" width="0.1524" layer="91"/>
+<wire x1="-144.78" y1="-177.8" x2="-167.64" y2="-177.8" width="0.1524" layer="91"/>
 <wire x1="-167.64" y1="-177.8" x2="-167.64" y2="-160.02" width="0.1524" layer="91"/>
-<pinref part="SELECTOR_PARAM_" gate="B" pin="A"/>
-<wire x1="-149.86" y1="-190.5" x2="-144.78" y2="-190.5" width="0.1524" layer="91"/>
-<wire x1="-149.86" y1="-177.8" x2="-149.86" y2="-190.5" width="0.1524" layer="91"/>
-<junction x="-149.86" y="-177.8"/>
 </segment>
 </net>
@@
 </segment>
 </net>
-<net name="N$5" class="0">
-<segment>
-<pinref part="SELECTOR_PARAM_" gate="B" pin="B"/>
-<wire x1="-152.4" y1="-193.04" x2="-144.78" y2="-193.04" width="0.1524" layer="91"/>
-<wire x1="-152.4" y1="-180.34" x2="-152.4" y2="-193.04" width="0.1524" layer="91"/>
-<wire x1="-170.18" y1="-180.34" x2="-152.4" y2="-180.34" width="0.1524" layer="91"/>
-<wire x1="-170.18" y1="-157.48" x2="-170.18" y2="-180.34" width="0.1524" layer="91"/>
-<pinref part="INSTRUCTION_MEMORY_2" gate="G$1" pin="11"/>
-<wire x1="-162.56" y1="-157.48" x2="-170.18" y2="-157.48" width="0.1524" layer="91"/>
-</segment>
-</net>
-<net name="N$10" class="0">
-<segment>
-<pinref part="SELECTOR_PARAM_" gate="B" pin="Y3"/>
-<wire x1="-60.96" y1="-175.26" x2="-40.64" y2="-175.26" width="0.1524" layer="91"/>
-<wire x1="-40.64" y1="-175.26" x2="-40.64" y2="-154.94" width="0.1524" layer="91"/>
-<wire x1="-40.64" y1="-154.94" x2="-50.8" y2="-154.94" width="0.1524" layer="91"/>
-<wire x1="-50.8" y1="-154.94" x2="-50.8" y2="-147.32" width="0.1524" layer="91"/>
-<wire x1="-50.8" y1="-147.32" x2="-2.54" y2="-147.32" width="0.1524" layer="91"/>
-<wire x1="73.66" y1="63.5" x2="73.66" y2="25.4" width="0.1524" layer="91"/>
-<wire x1="73.66" y1="25.4" x2="71.12" y2="25.4" width="0.1524" layer="91"/>
-<wire x1="71.12" y1="25.4" x2="71.12" y2="-30.48" width="0.1524" layer="91"/>
-<wire x1="71.12" y1="-30.48" x2="68.58" y2="-30.48" width="0.1524" layer="91"/>
-<wire x1="68.58" y1="-30.48" x2="68.58" y2="-114.3" width="0.1524" layer="91"/>
-<wire x1="68.58" y1="-114.3" x2="22.86" y2="-114.3" width="0.1524" layer="91"/>
-<wire x1="22.86" y1="-114.3" x2="22.86" y2="-124.46" width="0.1524" layer="91"/>
-<wire x1="22.86" y1="-124.46" x2="-2.54" y2="-124.46" width="0.1524" layer="91"/>
-<wire x1="-2.54" y1="-124.46" x2="-2.54" y2="-147.32" width="0.1524" layer="91"/>
-<wire x1="73.66" y1="63.5" x2="312.42" y2="63.5" width="0.1524" layer="91"/>
-<wire x1="312.42" y1="63.5" x2="312.42" y2="58.42" width="0.1524" layer="91"/>
-<pinref part="OUTPUT_BUFFER_KEYBOARD" gate="A" pin="G"/>
-<wire x1="312.42" y1="58.42" x2="317.5" y2="58.42" width="0.1524" layer="91"/>
-<wire x1="-119.38" y1="-198.12" x2="-93.98" y2="-198.12" width="0.1524" layer="91"/>
-<wire x1="-60.96" y1="-185.42" x2="-60.96" y2="-175.26" width="0.1524" layer="91"/>
-<wire x1="-93.98" y1="-198.12" x2="-93.98" y2="-185.42" width="0.1524" layer="91"/>
-<wire x1="-93.98" y1="-185.42" x2="-60.96" y2="-185.42" width="0.1524" layer="91"/>
-</segment>
-</net>
 <net name="N$26" class="1">
 <segment>
@@
 </segment>
 </net>
+<net name="N$5" class="0">
+<segment>
+<pinref part="SELECTOR_PARAM_" gate="B" pin="B"/>
+<pinref part="SELECTOR_INSRUCTION_LOWER" gate="A" pin="4Y"/>
+<wire x1="30.48" y1="30.48" x2="22.86" y2="30.48" width="0.1524" layer="91"/>
+</segment>
+</net>
+<net name="N$10" class="0">
+<segment>
+<pinref part="SELECTOR_INSRUCTION_LOWER" gate="A" pin="3Y"/>
+<pinref part="SELECTOR_PARAM_" gate="B" pin="A"/>
+<wire x1="22.86" y1="35.56" x2="22.86" y2="33.02" width="0.1524" layer="91"/>
+<wire x1="22.86" y1="33.02" x2="30.48" y2="33.02" width="0.1524" layer="91"/>
+</segment>
+</net>
+<net name="N$210" class="0">
+<segment>
+<pinref part="OUTPUT_BUFFER_KEYBOARD" gate="A" pin="G"/>
+<wire x1="312.42" y1="58.42" x2="317.5" y2="58.42" width="0.1524" layer="91"/>
+<wire x1="312.42" y1="63.5" x2="312.42" y2="58.42" width="0.1524" layer="91"/>
+<wire x1="73.66" y1="63.5" x2="312.42" y2="63.5" width="0.1524" layer="91"/>
+<wire x1="73.66" y1="63.5" x2="73.66" y2="25.4" width="0.1524" layer="91"/>
+<pinref part="SELECTOR_PARAM_" gate="B" pin="Y3"/>
+<wire x1="55.88" y1="25.4" x2="73.66" y2="25.4" width="0.1524" layer="91"/>
+</segment>
+</net>
