File: V5/Modules/Backplane/Backplane.brd (EAGLE design)
At the start: 97 x 98 mm, 23 parts, among them T1 2N3565, T2 2N3565, T3 2N3565, T4 2N3565

Commit message: update
Parts:
- removed NO_INVERT_JUMPER, NO_INVERT_JUMPER1, NO_INVERT_JUMPER2, NO_INVERT_JUMPER3: SSW-103-02-G-S, con-samtec:SSW-103-02-G-S
- removed R1, R2, R3, R4, R5, R6, R7, R8: ~220, rcl:0204/7
- removed SIGS_IN: SSW-106-02-G-D, con-samtec:SSW-106-02-G-D
- removed T1, T2, T3, T4: 2N3565, transistor:TO92
- added CLK_INV, CLR_INV, IN_INV, OUT_INV: SSW-103-02-G-S, con-samtec:SSW-103-02-G-S
- added IC1: 74AC04N, 74xx-eu:DIL14
- moved U$1 3.15 mm to (31.0, 38.0)
- moved ADDR_INCOMING 2.24 mm to (2.00, 25.0)
- moved ADDR_OUTGOING 1.48 mm to (88.4, 25.0)
- moved DB_OUTGOING 1.29 mm to (88.4, 73.0)
- moved DB_INCOMING 1.00 mm to (2.00, 73.0)
- moved RS_DATA 0.81 mm to (40.0, 48.0)
Connections:
- removed net N$1 (its old number): SIGS_IN.1, U$1.A31
- removed net N$11 (its old number): NO_INVERT_JUMPER1.2, R2.2, U$1.A28
- removed net N$12 (its old number): NO_INVERT_JUMPER1.3, R3.2, SIGS_IN.6, T2.1
- removed net N$13 (its old number): R4.1, T3.2
- removed net N$14 (its old number): NO_INVERT_JUMPER2.2, R4.2, U$1.A3
- removed net N$3 (its old number): SIGS_IN.3, U$1.A30
- removed net N$4 (its old number): SIGS_IN.5, U$1.A29
- removed net N$5 (its old number): SIGS_IN.7, U$1.B31
- removed net N$6 (its old number): SIGS_IN.9, U$1.B30
- removed net N$7 (its old number): SIGS_IN.11, U$1.B29
- new net N$25: CLR_INV.2, U$1.B28
- new net N$26: CLK_INV.2, U$1.A28
- new net N$27: IN_INV.2, U$1.A3
- new net N$28: OUT_INV.2, U$1.A2
- net GND: now also IC1.7; no longer SIGS_IN.2, T1.3, T2.3, T3.3, T4.3
- net N$10: now also IC1.9, OUT_INV.3; no longer R2.1, T2.2
- net N$15: now also CLR_INV.1, IC1.2; no longer NO_INVERT_JUMPER2.3, R5.2, SIGS_IN.8, T3.1
- net N$16: now also CLK_INV.1, IC1.4; no longer R6.1, T4.2
- net N$17: now also IC1.6, IN_INV.1; no longer NO_INVERT_JUMPER3.2, R6.2, U$1.A2
- net N$18: now also IC1.8, OUT_INV.1; no longer NO_INVERT_JUMPER3.3, R7.2, SIGS_IN.10, T4.1
- net N$2: now also CLR_INV.3, IC1.1; no longer R8.1, T1.2
- net N$8: now also CLK_INV.3, IC1.3; no longer NO_INVERT_JUMPER.2, R8.2, U$1.B28
- net N$9: now also IC1.5, IN_INV.3; no longer NO_INVERT_JUMPER.3, R1.2, SIGS_IN.4, T1.1
- net VCC: now also IC1.14; no longer R1.1, R3.1, R5.1, R7.1, SIGS_IN.12
Other:
- board size 97 x 98 mm -> 98 x 98 mm
