File: V5/Modules/Backplane/Backplane.sch (EAGLE design)
At the start: 23 parts, among them T1 2N3565, T2 2N3565, T3 2N3565, T4 2N3565

Commit message: update
Parts:
- removed NO_INVERT_JUMPER, NO_INVERT_JUMPER1, NO_INVERT_JUMPER2, NO_INVERT_JUMPER3: SSW-103-02-G-S, con-samtec:SSW-103-02-G-S
- removed R1, R2, R3, R4, R5, R6, R7, R8: ~220, rcl:R-US_0204/7
- removed SIGS_IN: SSW-106-02-G-D, con-samtec:SSW-106-02-G-D
- removed T1, T2, T3, T4: 2N3565, transistor:2N3565
- added CLK_INV, CLR_INV, IN_INV, OUT_INV: SSW-103-02-G-S, con-samtec:SSW-103-02-G-S
- added IC1: 74AC04N, 74xx-eu:74AC04N
Connections:
- removed net GND: SIGS_IN-2.1, T1.E, T2.E, T3.E, T4.E
- removed net N$1 (its old number): SIGS_IN-1.1, U$1G$1.GP1
- removed net N$11 (its old number): NO_INVERT_JUMPER1-2.1, R2.2, U$1G$1.CLK
- removed net N$12 (its old number): NO_INVERT_JUMPER1-3.1, R3.2, SIGS_IN-6.1, T2.C
- removed net N$13 (its old number): R4.1, T3.B
- removed net N$14 (its old number): NO_INVERT_JUMPER2-2.1, R4.2, U$1G$1.DB_IN
- removed net N$3 (its old number): SIGS_IN-3.1, U$1G$1.GP2
- removed net N$4 (its old number): SIGS_IN-5.1, U$1G$1.GP3
- removed net N$5 (its old number): SIGS_IN-7.1, U$1G$1.GP4
- removed net N$6 (its old number): SIGS_IN-9.1, U$1G$1.GP5
- removed net N$7 (its old number): SIGS_IN-11.1, U$1G$1.GP6
- removed net VCC: R1.1, R3.1, R5.1, R7.1, SIGS_IN-12.1
- new net N$25: CLR_INV-2.1, U$1G$1.CLEAR
- new net N$26: CLK_INV-2.1, U$1G$1.CLK
- new net N$27: IN_INV-2.1, U$1G$1.DB_IN
- new net N$28: OUT_INV-2.1, U$1G$1.DB_OUT
- net N$10: now also IC1D.I, OUT_INV-3.1; no longer R2.1, T2.B
- net N$15: now also CLR_INV-1.1, IC1A.O; no longer NO_INVERT_JUMPER2-3.1, R5.2, SIGS_IN-8.1, T3.C
- net N$16: now also CLK_INV-1.1, IC1B.O; no longer R6.1, T4.B
- net N$17: now also IC1C.O, IN_INV-1.1; no longer NO_INVERT_JUMPER3-2.1, R6.2, U$1G$1.DB_OUT
- net N$18: now also IC1D.O, OUT_INV-1.1; no longer NO_INVERT_JUMPER3-3.1, R7.2, SIGS_IN-10.1, T4.C
- net N$2: now also CLR_INV-3.1, IC1A.I; no longer R8.1, T1.B
- net N$8: now also CLK_INV-3.1, IC1B.I; no longer NO_INVERT_JUMPER-2.1, R8.2, U$1G$1.CLEAR
- net N$9: now also IC1C.I, IN_INV-3.1; no longer NO_INVERT_JUMPER-3.1, R1.2, SIGS_IN-4.1, T1.C
Other:
- note removed: "Signal"
- note removed: "~Signal"
