File: V5/Utils/singleInverter/singleInverter.sch (EAGLE design)
At the start: 12 parts, among them IC1 74AC04N, T3 2N3565

Commit message: update
Parts:
- removed ADDR_INCOMING, DB_INCOMING, RS_DATA: SSW-116-02-G-S, con-samtec:SSW-116-02-G-S
- removed ADDR_OUTGOING, DB_OUTGOING: SSW-116-02-G-S-RA, con-samtec:SSW-116-02-G-S-RA
- removed IC1: 74AC04N, 74xx-eu:74AC04N
- removed U$1: BACKPLATE_INTERFACEHEADER, Computer:BACKPLATE_INTERFACEHEADER
Connections:
- removed net ADDR0: ADDR_INCOMING-1.1, ADDR_OUTGOING-16.1, U$1G$1.ADDR_0
- removed net ADDR1: ADDR_INCOMING-2.1, ADDR_OUTGOING-15.1, U$1G$1.ADDR_1
- removed net ADDR10: ADDR_INCOMING-11.1, ADDR_OUTGOING-6.1, U$1G$1.ADDR_10
- removed net ADDR11: ADDR_INCOMING-12.1, ADDR_OUTGOING-5.1, U$1G$1.ADDR_11
- removed net ADDR12: ADDR_INCOMING-13.1, ADDR_OUTGOING-4.1, U$1G$1.ADDR_12
- removed net ADDR13: ADDR_INCOMING-14.1, ADDR_OUTGOING-3.1, U$1G$1.ADDR_13
- removed net ADDR14: ADDR_INCOMING-15.1, ADDR_OUTGOING-2.1, U$1G$1.ADDR_14
- removed net ADDR15: ADDR_INCOMING-16.1, ADDR_OUTGOING-1.1, U$1G$1.ADDR_15
- removed net ADDR2: ADDR_INCOMING-3.1, ADDR_OUTGOING-14.1, U$1G$1.ADDR_2
- removed net ADDR3: ADDR_INCOMING-4.1, ADDR_OUTGOING-13.1, U$1G$1.ADDR_3
- removed net ADDR4: ADDR_INCOMING-5.1, ADDR_OUTGOING-12.1, U$1G$1.ADDR_4
- removed net ADDR5: ADDR_INCOMING-6.1, ADDR_OUTGOING-11.1, U$1G$1.ADDR_5
- removed net ADDR6: ADDR_INCOMING-7.1, ADDR_OUTGOING-10.1, U$1G$1.ADDR_6
- removed net ADDR7: ADDR_INCOMING-8.1, ADDR_OUTGOING-9.1, U$1G$1.ADDR_7
- removed net ADDR8: ADDR_INCOMING-9.1, ADDR_OUTGOING-8.1, U$1G$1.ADDR_8
- removed net ADDR9: ADDR_INCOMING-10.1, ADDR_OUTGOING-7.1, U$1G$1.ADDR_9
- removed net DB0: DB_INCOMING-1.1, DB_OUTGOING-16.1, U$1G$1.DB_0
- removed net DB1: DB_INCOMING-2.1, DB_OUTGOING-15.1, U$1G$1.DB_1
- removed net DB10: DB_INCOMING-11.1, DB_OUTGOING-6.1, U$1G$1.DB_10
- removed net DB11: DB_INCOMING-12.1, DB_OUTGOING-5.1, U$1G$1.DB_11
- removed net DB12: DB_INCOMING-13.1, DB_OUTGOING-4.1, U$1G$1.DB_12
- removed net DB13: DB_INCOMING-14.1, DB_OUTGOING-3.1, U$1G$1.DB_13
- removed net DB14: DB_INCOMING-15.1, DB_OUTGOING-2.1, U$1G$1.DB_14
- removed net DB15: DB_INCOMING-16.1, DB_OUTGOING-1.1, U$1G$1.DB_15
- removed net DB2: DB_INCOMING-3.1, DB_OUTGOING-14.1, U$1G$1.DB_2
- removed net DB3: DB_INCOMING-4.1, DB_OUTGOING-13.1, U$1G$1.DB_3
- removed net DB4: DB_INCOMING-5.1, DB_OUTGOING-12.1, U$1G$1.DB_4
- removed net DB5: DB_INCOMING-6.1, DB_OUTGOING-11.1, U$1G$1.DB_5
- removed net DB6: DB_INCOMING-7.1, DB_OUTGOING-10.1, U$1G$1.DB_6
- removed net DB7: DB_INCOMING-8.1, DB_OUTGOING-9.1, U$1G$1.DB_7
- removed net DB8: DB_INCOMING-9.1, DB_OUTGOING-8.1, U$1G$1.DB_8
- removed net DB9: DB_INCOMING-10.1, DB_OUTGOING-7.1, U$1G$1.DB_9
- removed net N$1: SIGS_IN-1.1, U$1G$1.GP1
- removed net N$19: RS_DATA-1.1, U$1G$1.RSDATA_0
- removed net N$20: RS_DATA-2.1, U$1G$1.RSDATA_1
- removed net N$21: RS_DATA-3.1, U$1G$1.RSDATA_2
- removed net N$22: RS_DATA-4.1, U$1G$1.RSDATA_3
- removed net N$23: RS_DATA-5.1, U$1G$1.RSDATA_4
- removed net N$24: RS_DATA-6.1, U$1G$1.RSDATA_5
- removed net N$25: RS_DATA-7.1, U$1G$1.RSDATA_6
- removed net N$26: RS_DATA-8.1, U$1G$1.RSDATA_7
- removed net N$27: RS_DATA-9.1, U$1G$1.RSDATA_8
- removed net N$28: RS_DATA-10.1, U$1G$1.RSDATA_9
- removed net N$29: RS_DATA-11.1, U$1G$1.RSDATA_10
- removed net N$3: SIGS_IN-3.1, U$1G$1.GP2
- removed net N$30: RS_DATA-12.1, U$1G$1.RSDATA_11
- removed net N$31: RS_DATA-13.1, U$1G$1.RSDATA_12
- removed net N$32: RS_DATA-14.1, U$1G$1.RSDATA_13
- removed net N$33: RS_DATA-15.1, U$1G$1.RSDATA_14
- removed net N$34: RS_DATA-16.1, U$1G$1.RSDATA_15
- removed net N$4: SIGS_IN-5.1, U$1G$1.GP3
- removed net N$5: SIGS_IN-7.1, U$1G$1.GP4
- removed net N$6: SIGS_IN-9.1, U$1G$1.GP5
- removed net N$7: SIGS_IN-11.1, U$1G$1.GP6
- net GND: no longer SIGS_IN-2.1
- net VCC: no longer SIGS_IN-12.1
Other:
- note removed: "Incoming"
- note removed: "Outgoing"
